Commit message: updates ur5 urdf and more

File: manipulators/ur5/manipulator.urdf (robot description, URDF)
Before this commit: robot ur10, 11 links, 10 joints
Links:
- removed link base
- removed link ee_link
- removed link world
- added link dummy_root
- added link rg2_hand, mass 0.29881464108881906; visual mesh filename=file://meshes/visual/rg2/hand.dae
- added link rg2_leftfinger, mass 0.24059267945559043; visual mesh filename=file://meshes/visual/rg2/finger.dae
- added link rg2_rightfinger, mass 0.24059267945559043; visual mesh filename=file://meshes/visual/rg2/finger.dae
- link base_link: mass 4.0 -> 4.210389694173812; geometry visual mesh filename=file://meshes/visual/ur5/base.dae
- link forearm_link: mass 3.87 -> 4.210389694173812; geometry visual mesh filename=file://meshes/visual/ur5/forearm.dae
- link shoulder_link: mass 7.778 -> 2.6078628081050645; geometry visual mesh filename=file://meshes/visual/ur5/shoulder.dae
- link tool0: mass 0.0 -> None
- link upper_arm_link: mass 12.93 -> 9.034556202946057; geometry visual mesh filename=file://meshes/visual/ur5/upperarm.dae
- link wrist_1_link: mass 1.96 -> 0.8652783044597422; geometry visual mesh filename=file://meshes/visual/ur5/wrist1.dae
- link wrist_2_link: mass 1.96 -> 0.8652786866955592; geometry visual mesh filename=file://meshes/visual/ur5/wrist2.dae
- link wrist_3_link: mass 0.202 -> 0.23285976783205536; geometry visual mesh filename=file://meshes/visual/ur5/wrist3.dae
Joints:
- removed joint base_link-base_fixed_joint
- removed joint ee_fixed_joint
- removed joint world_joint
- removed joint wrist_3_link-tool0_fixed_joint
- added joint dummy_root_to_base: type fixed, parent dummy_root, child base_link, origin xyz=0 0 0 rpy=0 0 0
- added joint end_effector_frame_fixed_joint: type fixed, parent wrist_3_link, child tool0, origin xyz=0 0.275 0 rpy=-1.570796325 0 0
- added joint rg2_finger_joint1: type revolute, parent rg2_hand, child rg2_leftfinger, origin xyz=0.105 0.017 0 rpy=0 0 0, axis 0 0 1, limit lower=0.0 upper=1.18 effort=1000.6 velocity=1.57
- added joint rg2_finger_joint2: type revolute, parent rg2_hand, child rg2_rightfinger, origin xyz=0.105 -0.017 0 rpy=0 0 0, axis 0 0 -1, limit lower=0.0 upper=1.18 effort=1000.6 velocity=1.57
- added joint ur5_hand_joint: type fixed, parent wrist_3_link, child rg2_hand, origin xyz=0 0.0823 0 rpy=1.570796325 0 1.570796325
- joint elbow_joint: limit lower=-3.14159265359 upper=3.14159265359 effort=150.0 velocity=3.15 -> lower=-2.75 upper=2.75 effort=150 velocity=3.15; origin xyz=0.0 -0.1719 0.612 rpy=0.0 0.0 0.0 -> xyz=0 -0.1197 0.425 rpy=0 0 0
- joint shoulder_lift_joint: limit lower=-6.28318530718 upper=6.28318530718 effort=330.0 velocity=2.16 -> lower=-1.57 upper=1.57 effort=150 velocity=3.15; origin xyz=0.0 0.220941 0.0 rpy=0.0 1.57079632679 0.0 -> xyz=0 0.13585 0 rpy=0 0 0
- joint shoulder_pan_joint: limit lower=-6.28318530718 upper=6.28318530718 effort=330.0 velocity=2.16 -> lower=-3.141592654 upper=3.141592654 effort=150 velocity=3.15; origin xyz=0.0 0.0 0.1273 rpy=0.0 0.0 0.0 -> xyz=0 0 0.089159 rpy=0 0 0
- joint wrist_1_joint: limit lower=-6.28318530718 upper=6.28318530718 effort=54.0 velocity=3.2 -> lower=-6.28319 upper=6.28319 effort=28 velocity=3.2; origin xyz=0.0 0.0 0.5723 rpy=0.0 1.57079632679 0.0 -> xyz=0 0 0.39225 rpy=0 0 0
- joint wrist_2_joint: limit lower=-6.28318530718 upper=6.28318530718 effort=54.0 velocity=3.2 -> lower=-6.28319 upper=6.28319 effort=28 velocity=3.2; origin xyz=0.0 0.1149 0.0 rpy=0.0 0.0 0.0 -> xyz=0 0.093 0 rpy=0 0 0
- joint wrist_3_joint: limit lower=-6.28318530718 upper=6.28318530718 effort=54.0 velocity=3.2 -> lower=-6.28319 upper=6.28319 effort=28 velocity=3.2; origin xyz=0.0 0.0 0.1157 rpy=0.0 0.0 0.0 -> xyz=0 0 0.09465 rpy=0 0 0
